File: 0000.0120.kicad_pcb (KiCad board)
At the start: 2 copper layers, 132.5 x 36 mm, 26 parts, among them J1 Conn_01x06, J3 Conn_01x08, J4 Conn_01x12, J5 Conn_01x14

Commit message: Added two new 6 LED variants.
Parts:
- added D23: 3mm, LED_THT:LED_D3.0mm, F.Cu at (148.7, 118.0)
- added D24: 3mm, LED_THT:LED_D3.0mm, F.Cu at (148.7, 124.0)
- added D25: 3mm, LED_THT:LED_D3.0mm, F.Cu at (148.7, 142.0)
- added D26: 3mm, LED_THT:LED_D3.0mm, F.Cu at (148.7, 136.0)
- added D27: 3mm, LED_THT:LED_D3.0mm, F.Cu at (148.7, 148.0)
- added D28: 3mm, LED_THT:LED_D3.0mm, F.Cu at (148.7, 130.0)
- added D29: 3mm, LED_THT:LED_D3.0mm, F.Cu at (143.7, 74.0)
- added D30: 3mm, LED_THT:LED_D3.0mm, F.Cu at (143.7, 80.0)
- added D31: 3mm, LED_THT:LED_D3.0mm, F.Cu at (146.3, 86.0)
- added D32: 3mm, LED_THT:LED_D3.0mm, F.Cu at (146.3, 92.0)
- added D33: 3mm, LED_THT:LED_D3.0mm, F.Cu at (146.3, 98.0)
- added D34: 3mm, LED_THT:LED_D3.0mm, F.Cu at (146.3, 104.0)
- added J2: PH254, Connector_PinHeader_2.54mm:PinHeader_2x02_P2.54mm_Horizontal, B.Cu at (138.7, 98.0)
- added J6: PH254, Connector_PinHeader_2.54mm:PinHeader_2x04_P2.54mm_Horizontal, B.Cu at (138.7, 142.3)
- added J7: PH254, Connector_PinHeader_2.54mm:PinHeader_2x02_P2.54mm_Horizontal, B.Cu at (148.7, 98.3)
- J1: value Conn_01x06 -> PH254
- J3: value Conn_01x08 -> PH254
- J4: value Conn_01x12 -> PH254
- J5: value Conn_01x14 -> PH254
- moved D1 40.3 mm to (75.0, 57.0)
- moved D10 40.3 mm to (150.0, 30.0)
- moved D11 40.3 mm to (150.0, 60.0)
- moved D12 40.3 mm to (115.0, 57.0)
- moved D13 40.3 mm to (115.0, 51.0)
- moved D14 40.3 mm to (115.0, 45.0)
- moved D15 40.3 mm to (115.0, 33.0)
- moved D16 40.3 mm to (115.0, 39.0)
- moved D17 40.3 mm to (190.0, 60.0)
- moved D18 40.3 mm to (190.0, 54.0)
- moved D19 40.3 mm to (190.0, 48.0)
- moved D2 40.3 mm to (75.0, 51.0)
- moved D20 40.3 mm to (190.0, 30.0)
- moved D21 40.3 mm to (190.0, 36.0)
- moved D22 40.3 mm to (190.0, 42.0)
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Routing:
- net Net-(D23-K): track 0.00 -> 29.0 mm
- net Net-(D24-K): track 0.00 -> 25.2 mm
- net Net-(D29-K): track 0.00 -> 25.0 mm
- net Net-(D30-K): track 0.00 -> 23.8 mm
- net Net-(D28-K): track 0.00 -> 15.6 mm
- net Net-(D31-K): track 0.00 -> 15.0 mm
- net Net-(D26-K): track 0.00 -> 13.0 mm
- net Net-(D32-K): track 0.00 -> 8.09 mm
- net Net-(D34-K): track 0.00 -> 6.29 mm
- net Net-(D27-K): track 0.00 -> 5.81 mm
- net Net-(D33-K): track 0.00 -> 4.98 mm
- net Net-(D25-K): track 0.00 -> 2.49 mm
- added copper zone on B.Cu, net Net-(D23-A)
- added copper zone on F.Cu, net Net-(D23-A)
- added copper zone on B.Cu, net Net-(D29-A)
- added copper zone on F.Cu, net Net-(D29-A)
Other:
- board size 132.5 x 36 mm -> 132.5 x 124 mm
