File: 0000.0120.kicad_sch (KiCad schematic)
At the start: 26 parts, among them J1 PH254, J3 PH254, J4 PH254, J5 PH254

Commit message: Added two new 6 LED variants.
Other:
- added sheet 6xVertical (6xV_1.kicad_sch)
- added sheet 6xVertical1 (6xV_2.kicad_sch)
